File: hardware/AK-280.kicad_sch (KiCad schematic)
At the start: 76 parts, among them J1 AUX, J101 AUDIO INPUT L, J2 BTL, J201 AUDIO INPUT R, J3 POWER DC 12V/5A, J4 POWER, P4 To Power Switch, SW1 POWER, U1 KIA 4558P, U2 KIA 4558P

Commit message: Add files via upload
Parts:
- added C6: 220μ, symbol Device:C_Polarized_Small
- AMP1: MANUFACTURER MCM Electronics -> Wuxi Youda Electronics
- C1: value 3300μ/16V -> 3300μ; Type (none) -> Aluminum Electrolytic (Standard); Voltage (none) -> 16V
- C101, C104, C201, C204: value 1μ/50V -> 1μ; Type (none) -> Aluminum Electrolytic (Low ESR); Voltage (none) -> 50V
- C102, C202: value 10μ/50V -> 10μ; Type (none) -> Aluminum Electrolytic (Low ESR); Voltage (none) -> 50V
- C103, C108, C203, C208: Type (none) -> Ceramic Capacitor (C0G)
- C105, C106, C107, C205, C206, C207: Type (none) -> Film Capacitor
- C109, C209: value 0.33μ/50V -> 0.33μ; Type (none) -> Aluminum Electrolytic (Low ESR); Voltage (none) -> 50V
- C2, C3: value 47μ/25V -> 47μ; Type (none) -> Aluminum Electrolytic (Standard); Voltage (none) -> 25V
- C4: value 220μ/16V -> 220μ; Type (none) -> Aluminum Electrolytic (Standard); Voltage (none) -> 16V
- C5: Type (none) -> Ceramic Capacitor (X7R)
- D4: value Zener9.1V -> Zener; Voltage (none) -> 9.1V
- R1: value 10kΩ -> 10k; Wattage (none) -> 1/4W
- R101, R102, R103, R104, R105, R106, R107, R108, R109, R110, R111, R112, R113, R114, R201, R202, R203, R204, R205, R206, R207, R208, R209, R210, R211, R212, R213, R214, R3, R4, R5: Wattage (none) -> 1/4W
- R2: value 220 1/2W -> 220; Wattage (none) -> 1/2W
- U1, U2: MANUFACTURER (none) -> Korea Electronics
Connections:
- net GND: now also C6.2
- net at C102.2, C202.2, R106.1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: now also C6.1
